File: project/_driver.kicad_sch (KiCad schematic)
At the start: 18 parts, among them U201 74HC595

Commit message: fixing project info in all sheets
Other:
- title: WormControl-Relay15x5t15-ControlUI -> WormControl-Input32-UIBoard
Changed lines of the file:
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@@
   (paper "A4")
   (title_block
-    (title "WormControl-Relay15x5t15-ControlUI")
-    (date "2024-12-19")
+    (title "WormControl-Input32-UIBoard")
+    (date "2026-02-10")
     (rev "0.1")
     (company "makerspace.lt")

Commit message: updating kibot,fixing silkscreen, lowering led current
Parts:
- R201, R202, R203, R204, R205, R206, R207, R208: value 220R -> 330R; lcsc# C25091 -> C25104
Changed lines of the file:
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@@
     (in_bom yes) (on_board yes)
     (property "Reference" "R206" (id 0) (at 148.59 74.93 90))
-    (property "Value" "220R" (id 1) (at 143.51 76.2 90))
+    (property "Value" "330R" (id 1) (at 143.51 76.2 90))
     (property "Footprint" "Resistor_SMD:R_0402_1005Metric_Pad0.72x0.64mm_HandSolder" (id 2) (at 143.51 74.422 90)
       (effects (font (size 1.27 1.27)) hide)
@@
       (effects (font (size 1.27 1.27)) hide)
     )
-    (property "lcsc#" "C25091" (id 5) (at 143.51 76.2 0)
+    (property "lcsc#" "C25104" (id 5) (at 143.51 76.2 0)
       (effects (font (size 1.27 1.27)) hide)
     )
@@
     (in_bom yes) (on_board yes)
     (property "Reference" "R205" (id 0) (at 148.59 69.85 90))
-    (property "Value" "220R" (id 1) (at 143.51 71.12 90))
+    (property "Value" "330R" (id 1) (at 143.51 71.12 90))
     (property "Footprint" "Resistor_SMD:R_0402_1005Metric_Pad0.72x0.64mm_HandSolder" (id 2) (at 143.51 69.342 90)
       (effects (font (size 1.27 1.27)) hide)
@@
       (effects (font (size 1.27 1.27)) hide)
     )
-    (property "lcsc#" "C25091" (id 5) (at 143.51 71.12 0)
+    (property "lcsc#" "C25104" (id 5) (at 143.51 71.12 0)
       (effects (font (size 1.27 1.27)) hide)
     )
@@
     (in_bom yes) (on_board yes)
     (property "Reference" "R201" (id 0) (at 138.43 67.31 90))
-    (property "Value" "220R" (id 1) (at 133.35 68.58 90))
+    (property "Value" "330R" (id 1) (at 133.35 68.58 90))
     (property "Footprint" "Resistor_SMD:R_0402_1005Metric_Pad0.72x0.64mm_HandSolder" (id 2) (at 133.35 66.802 90)
       (effects (font (size 1.27 1.27)) hide)
@@
       (effects (font (size 1.27 1.27)) hide)
     )
-    (property "lcsc#" "C25091" (id 5) (at 133.35 68.58 0)
+    (property "lcsc#" "C25104" (id 5) (at 133.35 68.58 0)
       (effects (font (size 1.27 1.27)) hide)
     )
@@
     (in_bom yes) (on_board yes)
     (property "Reference" "R208" (id 0) (at 148.59 85.09 90))
-    (property "Value" "220R" (id 1) (at 143.51 86.36 90))
+    (property "Value" "330R" (id 1) (at 143.51 86.36 90))
     (property "Footprint" "Resistor_SMD:R_0402_1005Metric_Pad0.72x0.64mm_HandSolder" (id 2) (at 143.51 84.582 90)
       (effects (font (size 1.27 1.27)) hide)
@@
       (effects (font (size 1.27 1.27)) hide)
     )
-    (property "lcsc#" "C25091" (id 5) (at 143.51 86.36 0)
+    (property "lcsc#" "C25104" (id 5) (at 143.51 86.36 0)
       (effects (font (size 1.27 1.27)) hide)
     )
@@
     (in_bom yes) (on_board yes)
     (property "Reference" "R207" (id 0) (at 148.59 80.01 90))
-    (property "Value" "220R" (id 1) (at 143.51 81.28 90))
+    (property "Value" "330R" (id 1) (at 143.51 81.28 90))
     (property "Footprint" "Resistor_SMD:R_0402_1005Metric_Pad0.72x0.64mm_HandSolder" (id 2) (at 143.51 79.502 90)
       (effects (font (size 1.27 1.27)) hide)
@@
       (effects (font (size 1.27 1.27)) hide)
     )
-    (property "lcsc#" "C25091" (id 5) (at 143.51 81.28 0)
+    (property "lcsc#" "C25104" (id 5) (at 143.51 81.28 0)
       (effects (font (size 1.27 1.27)) hide)
     )
@@
     (in_bom yes) (on_board yes)
     (property "Reference" "R203" (id 0) (at 138.43 77.47 90))
-    (property "Value" "220R" (id 1) (at 133.35 78.74 90))
+    (property "Value" "330R" (id 1) (at 133.35 78.74 90))
     (property "Footprint" "Resistor_SMD:R_0402_1005Metric_Pad0.72x0.64mm_HandSolder" (id 2) (at 133.35 76.962 90)
       (effects (font (size 1.27 1.27)) hide)
@@
       (effects (font (size 1.27 1.27)) hide)
     )
-    (property "lcsc#" "C25091" (id 5) (at 133.35 78.74 0)
+    (property "lcsc#" "C25104" (id 5) (at 133.35 78.74 0)
       (effects (font (size 1.27 1.27)) hide)
     )
@@
     (in_bom yes) (on_board yes)
     (property "Reference" "R202" (id 0) (at 138.43 72.39 90))
-    (property "Value" "220R" (id 1) (at 133.35 73.66 90))
+    (property "Value" "330R" (id 1) (at 133.35 73.66 90))
     (property "Footprint" "Resistor_SMD:R_0402_1005Metric_Pad0.72x0.64mm_HandSolder" (id 2) (at 133.35 71.882 90)
       (effects (font (size 1.27 1.27)) hide)
@@
       (effects (font (size 1.27 1.27)) hide)
     )
-    (property "lcsc#" "C25091" (id 5) (at 133.35 73.66 0)
+    (property "lcsc#" "C25104" (id 5) (at 133.35 73.66 0)
       (effects (font (size 1.27 1.27)) hide)
     )
@@
     (in_bom yes) (on_board yes)
     (property "Reference" "R204" (id 0) (at 138.43 82.55 90))
-    (property "Value" "220R" (id 1) (at 133.35 83.82 90))
+    (property "Value" "330R" (id 1) (at 133.35 83.82 90))
     (property "Footprint" "Resistor_SMD:R_0402_1005Metric_Pad0.72x0.64mm_HandSolder" (id 2) (at 133.35 82.042 90)
       (effects (font (size 1.27 1.27)) hide)
@@
       (effects (font (size 1.27 1.27)) hide)
     )
-    (property "lcsc#" "C25091" (id 5) (at 133.35 83.82 0)
-      (effects (font (size 1.27 1.27)) hide)
-    )
+    (property "lcsc#" "C25104" (id 5) (at 133.35 83.82 0)
+      (effects (font (size 1.27 1.27)) hide)
+    )

Commit message: parts consolidation and small fixes
* Inverting input LEDs
* Switching to TMP102 as TMP101 is no longer available
* Helping 74HC forget state after power loss
* bumping up version
Connections:
- net Ar: now also D201.1 (K); no longer D201.2 (A)
- net Br: now also D205.1 (K); no longer D205.2 (A)
- net Cr: now also D202.1 (K); no longer D202.2 (A)
- net Dr: now also D206.1 (K); no longer D206.2 (A)
- net Er: now also D203.1 (K); no longer D203.2 (A)
- net Fr: now also D207.1 (K); no longer D207.2 (A)
- net GND: no longer D201.1 (K), D202.1 (K), D203.1 (K), D204.1 (K), D205.1 (K), D206.1 (K), D207.1 (K), D208.1 (K)
- net Gr: now also D204.1 (K); no longer D204.2 (A)
- net Hr: now also D208.1 (K); no longer D208.2 (A)
- net Vcc: now also D201.2 (A), D202.2 (A), D203.2 (A), D204.2 (A), D205.2 (A), D206.2 (A), D207.2 (A), D208.2 (A)
Other:
- moved on the sheet: D201, D202, D203, D204, D205, D206, D207, D208
Changed lines of the file:
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@@
   (title_block
     (title "WormControl-Input32-UIBoard")
-    (date "2026-02-10")
-    (rev "0.1")
+    (date "2026-03-19")
+    (rev "0.2")
     (company "makerspace.lt")
   )
@@
   (hierarchical_label "Vcc" (shape input) (at 114.3 60.96 180)
     (effects (font (size 1.27 1.27)) (justify right))
-  )
-  (hierarchical_label "GND" (shape bidirectional) (at 184.15 86.36 0)
-    (effects (font (size 1.27 1.27)) (justify left))
   )
   (hierarchical_label "DATA_OUT" (shape output) (at 124.46 91.44 0)
@@
     (effects (font (size 1.27 1.27)) (justify right))
   )
+  (hierarchical_label "Vcc" (shape input) (at 184.15 86.36 0)
+    (effects (font (size 1.27 1.27)) (justify left))
+  )
   (hierarchical_label "GND" (shape bidirectional) (at 123.19 60.96 0)
     (effects (font (size 1.27 1.27)) (justify left))
@@
     (effects (font (size 1.27 1.27)) (justify right))
   )
-  (symbol (lib_id "Device:LED") (at 161.29 83.82 180) (unit 1)
-    (in_bom yes) (on_board yes)
-    (property "Reference" "D204" (id 0) (at 157.48 82.55 0))
-    (property "Value" "RED" (id 1) (at 157.48 85.09 0))
+  (symbol (lib_id "Device:LED") (at 161.29 83.82 0) (unit 1)
+    (in_bom yes) (on_board yes)
+    (property "Reference" "D204" (id 0) (at 165.1 85.09 0))
+    (property "Value" "RED" (id 1) (at 165.1 82.55 0))
     (property "Footprint" "-local:LED_1206_3216Metric_ReverseMount" (id 2) (at 161.29 83.82 0)
       (effects (font (size 1.27 1.27)) hide)
@@
     (pin "2")
   )
-  (symbol (lib_id "Device:LED") (at 161.29 68.58 180) (unit 1)
-    (in_bom yes) (on_board yes)
-    (property "Reference" "D201" (id 0) (at 157.48 67.31 0))
-    (property "Value" "RED" (id 1) (at 157.48 69.85 0))
+  (symbol (lib_id "Device:LED") (at 161.29 68.58 0) (unit 1)
+    (in_bom yes) (on_board yes)
+    (property "Reference" "D201" (id 0) (at 165.1 69.85 0))
+    (property "Value" "RED" (id 1) (at 165.1 67.31 0))
     (property "Footprint" "-local:LED_1206_3216Metric_ReverseMount" (id 2) (at 161.29 68.58 0)
       (effects (font (size 1.27 1.27)) hide)
@@
     (pin "2")
   )
-  (symbol (lib_id "Device:LED") (at 172.72 81.28 180) (unit 1)
-    (in_bom yes) (on_board yes)
-    (property "Reference" "D207" (id 0) (at 168.91 80.01 0))
-    (property "Value" "RED" (id 1) (at 168.91 82.55 0))
+  (symbol (lib_id "Device:LED") (at 172.72 81.28 0) (unit 1)
+    (in_bom yes) (on_board yes)
+    (property "Reference" "D207" (id 0) (at 176.53 82.55 0))
+    (property "Value" "RED" (id 1) (at 176.53 80.01 0))
     (property "Footprint" "-local:LED_1206_3216Metric_ReverseMount" (id 2) (at 172.72 81.28 0)
       (effects (font (size 1.27 1.27)) hide)
@@
     (pin "2")
   )
-  (symbol (lib_id "Device:LED") (at 172.72 76.2 180) (unit 1)
-    (in_bom yes) (on_board yes)
-    (property "Reference" "D206" (id 0) (at 168.91 74.93 0))
-    (property "Value" "RED" (id 1) (at 168.91 77.47 0))
+  (symbol (lib_id "Device:LED") (at 172.72 76.2 0) (unit 1)
+    (in_bom yes) (on_board yes)
+    (property "Reference" "D206" (id 0) (at 176.53 77.47 0))
+    (property "Value" "RED" (id 1) (at 176.53 74.93 0))
     (property "Footprint" "-local:LED_1206_3216Metric_ReverseMount" (id 2) (at 172.72 76.2 0)
       (effects (font (size 1.27 1.27)) hide)
@@
     (pin "2")
   )
-  (symbol (lib_id "Device:LED") (at 172.72 86.36 180) (unit 1)
-    (in_bom yes) (on_board yes)
-    (property "Reference" "D208" (id 0) (at 168.91 85.09 0))
-    (property "Value" "RED" (id 1) (at 168.91 87.63 0))
+  (symbol (lib_id "Device:LED") (at 172.72 86.36 0) (unit 1)
+    (in_bom yes) (on_board yes)
+    (property "Reference" "D208" (id 0) (at 176.53 87.63 0))
+    (property "Value" "RED" (id 1) (at 176.53 85.09 0))
     (property "Footprint" "-local:LED_1206_3216Metric_ReverseMount" (id 2) (at 172.72 86.36 0)
       (effects (font (size 1.27 1.27)) hide)
@@
     (pin "9")
   )
-  (symbol (lib_id "Device:LED") (at 161.29 78.74 180) (unit 1)
-    (in_bom yes) (on_board yes)
-    (property "Reference" "D203" (id 0) (at 157.48 77.47 0))
-    (property "Value" "RED" (id 1) (at 157.48 80.01 0))
+  (symbol (lib_id "Device:LED") (at 161.29 78.74 0) (unit 1)
+    (in_bom yes) (on_board yes)
+    (property "Reference" "D203" (id 0) (at 165.1 80.01 0))
+    (property "Value" "RED" (id 1) (at 165.1 77.47 0))
     (property "Footprint" "-local:LED_1206_3216Metric_ReverseMount" (id 2) (at 161.29 78.74 0)
       (effects (font (size 1.27 1.27)) hide)
@@
     (pin "2")
   )
-  (symbol (lib_id "Device:LED") (at 161.29 73.66 180) (unit 1)
-    (in_bom yes) (on_board yes)
-    (property "Reference" "D202" (id 0) (at 157.48 72.39 0))
-    (property "Value" "RED" (id 1) (at 157.48 74.93 0))
+  (symbol (lib_id "Device:LED") (at 161.29 73.66 0) (unit 1)
+    (in_bom yes) (on_board yes)
+    (property "Reference" "D202" (id 0) (at 165.1 74.93 0))
+    (property "Value" "RED" (id 1) (at 165.1 72.39 0))
     (property "Footprint" "-local:LED_1206_3216Metric_ReverseMount" (id 2) (at 161.29 73.66 0)
       (effects (font (size 1.27 1.27)) hide)
@@
     (pin "2")
   )
-  (symbol (lib_id "Device:LED") (at 172.72 71.12 180) (unit 1)
-    (in_bom yes) (on_board yes)
-    (property "Reference" "D205" (id 0) (at 168.91 69.85 0))
-    (property "Value" "RED" (id 1) (at 168.91 72.39 0))
+  (symbol (lib_id "Device:LED") (at 172.72 71.12 0) (unit 1)
+    (in_bom yes) (on_board yes)
+    (property "Reference" "D205" (id 0) (at 176.53 72.39 0))
+    (property "Value" "RED" (id 1) (at 176.53 69.85 0))
     (property "Footprint" "-local:LED_1206_3216Metric_ReverseMount" (id 2) (at 172.72 71.12 0)
       (effects (font (size 1.27 1.27)) hide)
